File: Circuit/MotorcycleSpeedo/MotorcycleSpeedo.sch (KiCad schematic (older format))
At the start: 50 parts

Commit message: made some schematic changes, close to finishing and getting ready to send it to fab
Parts:
- removed C? (x2): C, symbol Device:C
- removed D?: D_TVS, symbol Device:D_TVS
- removed D?: D_TVS_x2_AAC, symbol Device:D_TVS_x2_AAC
- removed JP? (x2): Jumper_3_Bridged12, symbol Jumper:Jumper_3_Bridged12
- removed R? (x3): R, symbol Device:R
- removed U?: MAX31855KASA, Package_SO:SOIC-8_3.9x4.9mm_P1.27mm, symbol Sensor_Temperature:MAX31855KASA
- added C101, C102: 0.1uF, Capacitor_SMD:C_0805_2012Metric, symbol Device:C
- added C103, C104: 0.22uF, Capacitor_SMD:C_0805_2012Metric, symbol Device:C
- added C107, C108: C, Capacitor_SMD:C_0805_2012Metric, symbol Device:C
- added D105: SP721, symbol SP721:SP721
- added R101, R102: 2.49K, Resistor_SMD:R_0603_1608Metric, symbol Device:R
- added R103, R106: 470, Resistor_SMD:R_0603_1608Metric, symbol Device:R
- added R107, R108, R109: R, symbol Device:R
- added U103: L7805, symbol Regulator_Linear:L7805
- added U104: 1602LCD, symbol 1602I2C:1602LCD
- BT101: renamed from BT?; footprint (none) -> Battery:BatteryHolder_Keystone_1060_1x2032
- C105, C106, C109, C110: renamed from C?; footprint (none) -> Capacitor_SMD:C_0805_2012Metric
- D101, D102, D104, D107, D109, D110, D111, D112: renamed from D?; footprint (none) -> Package_TO_SOT_SMD:SOT-23; Manufacturer PN (none) -> MMBD7000LT1G
- D116: renamed from D?; value LEFT -> NEUTRAL
- gave numbers to parts that had none: 26
Connections:
- net labels added: RPM_OUT, TEMP1+, TEMP1-, TEMP1_OUT, TEMP2+, TEMP2-, TEMP2_OUT, TVS1, TVS2, TVS3, TVS4, TVS5, TVS6
- net labels removed: +3V3, TEMP+, TEMP-, TEMP_THERMISTOR_OUT
- wire segments 149 -> 178
Other:
- note added: "NOTE! CHECK THE RESISTOR VALUES!!!\n"

Commit message: Board built enough to submit. I'm sure changes will be made.
Parts:
- removed A101: Arduino_Nano_v3.x, Module:Arduino_Nano, symbol MCU_Module:Arduino_Nano_v3.x
- removed D101, D102, D104, D107, D109, D110, D111, D112: D_x2_Serial_ACK, Package_TO_SOT_SMD:SOT-23, symbol Device:D_x2_Serial_ACK
- removed U101: LTV-817, Package_DIP:DIP-4_W7.62mm, symbol Isolator:LTV-817
- removed U103: L7805, symbol Regulator_Linear:L7805
- removed U104: 1602LCD, symbol 1602I2C:1602LCD
- removed U105: MCP7940N-xSN, symbol Timer:MCP7940N-xSN
- added C103, C104, C108, C110, C113, C117, C118, C119, C120, C121, C122, C123, C124, C125, C126, C127, C132, C133, C145: C, Capacitor_SMD:C_0603_1608Metric, symbol Device:C
- added C105, C134, C137, C138, C139, C143, C144: .1uF, Capacitor_SMD:C_0603_1608Metric, symbol Device:C
- added C109, C111, C112: .1uf, Capacitor_SMD:C_0603_1608Metric, symbol Device:C
- added C114: 100uF, Capacitor_SMD:C_0603_1608Metric, symbol Device:CP
- added C115: 1500pf, Capacitor_SMD:C_0603_1608Metric, symbol Device:C
- added C116: CP, Capacitor_SMD:C_0603_1608Metric, symbol Device:CP
- added C128, C129: 20pF, Capacitor_SMD:C_0603_1608Metric, symbol Device:C
- added C142: .01uF, Capacitor_SMD:C_0603_1608Metric, symbol Device:C
- added D105, D106, D107, D108, D109, D110, D111, D112, D113, D114, D115, D116, D117, D118, D120, D121, D123, D124, D125, D126, D127, D128, D129, D130: LED, LED_SMD:LED_0603_1608Metric_Pad1.05x0.95mm_HandSolder, symbol Device:LED
- added D119, D122, D131: D, Diode_SMD:D_SMA, symbol Device:D
- added H101, H102, H103, H104, H105, H106: MountingHole_Pad, MountingHole:MountingHole_3.2mm_M3_DIN965_Pad, symbol Mechanical:MountingHole_Pad
- added J101: Conn_01x07_Female, Connector_PinHeader_2.54mm:PinHeader_1x07_P2.54mm_Vertical, symbol Connector:Conn_01x07_Female
- added J102, J104, J107: Conn_01x03_Female, Connector_PinHeader_2.54mm:PinHeader_1x03_P2.54mm_Vertical, symbol Connector:Conn_01x03_Female
- added J103: Conn_01x02_Female, Connector_PinHeader_2.54mm:PinHeader_1x02_P2.54mm_Vertical, symbol Connector:Conn_01x02_Female
- added J105, J109: Conn_01x04_Female, Connector_PinHeader_2.54mm:PinHeader_1x04_P2.54mm_Vertical, symbol Connector:Conn_01x04_Female
- added J106: Conn_02x04_Counter_Clockwise, Connector_PinHeader_2.54mm:PinHeader_2x04_P2.54mm_Vertical, symbol Connector_Generic:Conn_02x04_Odd_Even
- added J108: Conn_01x04_Male, Connector_PinHeader_1.27mm:PinHeader_1x04_P1.27mm_Vertical, symbol Connector:Conn_01x04_Male
- added J110: Conn_01x01_Female, TestPoint:TestPoint_Pad_1.5x1.5mm, symbol Connector:Conn_01x01_Female
- added JP101, JP102, JP103: SolderJumper_3_Bridged12, Jumper:SolderJumper-3_P1.3mm_Bridged12_Pad1.0x1.5mm_NumberLabels, symbol Jumper:SolderJumper_3_Bridged12
- added L101: 220, MotorcycleSpeedo:SMSD0804-Inductor, symbol Device:L
- added Q101, Q102, Q104: Q_NMOS_GSD, Package_TO_SOT_SMD:SOT-23, symbol Device:Q_NMOS_GSD
- added Q103: Q_PMOS_GSD, Package_TO_SOT_SMD:SOT-23, symbol Device:Q_PMOS_GSD
- added R102, R103, R105, R106, R113, R114, R116, R117, R118, R119, R121, R122, R123, R127, R128, R130: R, Resistor_SMD:R_0603_1608Metric, symbol Device:R
- added R107, R112, R124, R131, R133, R134, R135, R136, R140: 10K, Resistor_SMD:R_0603_1608Metric, symbol Device:R
- added R109: 470, Resistor_SMD:R_0603_1608Metric, symbol Device:R
- added R115: 180, Resistor_SMD:R_0603_1608Metric, symbol Device:R
- added R120: 120, Resistor_SMD:R_0603_1608Metric, symbol Device:R
- added R129, R141: 1k, Resistor_SMD:R_0603_1608Metric, symbol Device:R
- added R146, R147, R148, R149, R150: 560, Resistor_SMD:R_0603_1608Metric, symbol Device:R
- added R151, R152: 22, Resistor_SMD:R_0603_1608Metric, symbol Device:R
- added U101: AP131-33, Package_TO_SOT_SMD:SOT-23-5, symbol Regulator_Linear:AP131-33
- added U103: APT8L08, Package_SO:SOIC-14_3.9x8.7mm_P1.27mm, symbol APT8L08:APT8L08
- added U104: BMP280, Package_LGA:Bosch_LGA-8_2x2.5mm_P0.65mm_ClockwisePinNumbering, symbol Sensor_Pressure:BMP280
- added U105: MPU-9250, Sensor_Motion:InvenSense_QFN-24_3x3mm_P0.4mm, symbol Sensor_Motion:MPU-9250
- added U106: LTV-817, Package_DIP:DIP-4_W7.62mm, symbol Isolator:LTV-817
- added U107: MC34063AD, Package_SO:SOIC-8_3.9x4.9mm_P1.27mm, symbol Regulator_Switching:MC34063AD
- added U108: TJA1051T-E, Package_SO:SOIC-8_3.9x4.9mm_P1.27mm, symbol Interface_CAN_LIN:TJA1051T-E
- added U110: FM116B, Package_TO_SOT_SMD:SOT-23-6, symbol FM116:FM116B
- added U111: 74AHCT1G14, Package_TO_SOT_SMD:SOT-353_SC-70-5, symbol 74xGxx:74AHCT1G14
- added U112: STM32F103C8Tx, Package_QFP:LQFP-48_7x7mm_P0.5mm, symbol MCU_ST_STM32F1:STM32F103C8Tx
- added U113: TC1508S, Package_SO:SOP-16_4.55x10.3mm_P1.27mm, symbol TC1509S:TC1509S
- added U114: TC1509S, Package_SO:SOP-16_4.55x10.3mm_P1.27mm, symbol TC1509S:TC1509S
- added U1[2: AMS1117-5.0, Package_TO_SOT_SMD:SOT-223, symbol Regulator_Linear:AMS1117-5.0
- added V101, V103: HV5812, Package_SO:SOIC-28W_7.5x17.9mm_P1.27mm, symbol HV5812:HV5812
- added V102: HNA-12MM54T, HNA-12MM54T_VFD:HNA-12MM54T, symbol HNA-12MM54T:HNA-12MM54T
- added Y101: 8M, Crystal:Crystal_SMD_5032-2Pin_5.0x3.2mm, symbol Device:Crystal
- BT101: Manufacturer PN (none) -> CR2032-BS-6-1
- C101: renamed from C105; footprint Capacitor_SMD:C_0805_2012Metric -> Capacitor_SMD:C_0603_1608Metric
- C102: renamed from C106; footprint Capacitor_SMD:C_0805_2012Metric -> Capacitor_SMD:C_0603_1608Metric
- C106: renamed from C107; footprint Capacitor_SMD:C_0805_2012Metric -> Capacitor_SMD:C_0603_1608Metric
- C107: renamed from C108; footprint Capacitor_SMD:C_0805_2012Metric -> Capacitor_SMD:C_0603_1608Metric
- C130: renamed from C110; footprint Capacitor_SMD:C_0805_2012Metric -> Capacitor_SMD:C_0603_1608Metric
- C131: renamed from C109; footprint Capacitor_SMD:C_0805_2012Metric -> Capacitor_SMD:C_0603_1608Metric
- C135: renamed from C102; footprint Capacitor_SMD:C_0805_2012Metric -> Capacitor_SMD:C_0603_1608Metric
- C136: renamed from C104; footprint Capacitor_SMD:C_0805_2012Metric -> Capacitor_SMD:C_0603_1608Metric
- C140: renamed from C101; footprint Capacitor_SMD:C_0805_2012Metric -> Capacitor_SMD:C_0603_1608Metric
- C141: renamed from C103; footprint Capacitor_SMD:C_0805_2012Metric -> Capacitor_SMD:C_0603_1608Metric
- D101: renamed from D108; footprint (none) -> Diode_SMD:D_SMA
- D102: renamed from D103; footprint (none) -> Diode_SMD:D_SMA
- D103: renamed from D106; footprint (none) -> Diode_SMD:D_SMA
- D104: renamed from D105; footprint (none) -> Package_SO:SOIC-8_3.9x4.9mm_P1.27mm
- D132: renamed from D113; footprint (none) -> Indicators:HF.SilkSF.Cu
- D133: renamed from D114; footprint (none) -> Indicators:RightPointingF.SilkSF.Cu
- D134: renamed from D115; footprint (none) -> Indicators:LeftPointingF.SilkSF.Cu
- D135: renamed from D116; footprint (none) -> Indicators:NF.SilkSF.Cu
- F101: footprint (none) -> Fuse:Fuse_1206_3216Metric; Manufacturer PN (none) -> JK-NSMD100-16V
- JP104: renamed from JP101; footprint (none) -> Jumper:SolderJumper-3_P1.3mm_Bridged12_RoundedPad1.0x1.5mm_NumberLabels
- JP105: renamed from JP102; footprint (none) -> Jumper:SolderJumper-3_P1.3mm_Bridged12_RoundedPad1.0x1.5mm_NumberLabels
- JP106: renamed from JP103; footprint (none) -> Jumper:SolderJumper-3_P1.3mm_Bridged12_RoundedPad1.0x1.5mm_NumberLabels
- JP107: renamed from JP104; footprint (none) -> Jumper:SolderJumper-3_P1.3mm_Bridged12_RoundedPad1.0x1.5mm_NumberLabels
- M101, M102: footprint (none) -> X25Stepper:x25FrontStepper
- R101: renamed from R109; footprint (none) -> Resistor_SMD:R_0603_1608Metric
- R104, R108: footprint (none) -> Resistor_SMD:R_0603_1608Metric
- R110: value R -> 10K; footprint (none) -> Resistor_SMD:R_0603_1608Metric
- R111: value R -> .22; footprint (none) -> Resistor_SMD:R_0603_1608Metric
- R125: renamed from R107; value R -> 10K; footprint (none) -> Resistor_SMD:R_0603_1608Metric
- R126: renamed from R105; footprint (none) -> Resistor_SMD:R_0603_1608Metric
- R132: renamed from R112; footprint (none) -> Resistor_SMD:R_0603_1608Metric
- R137: renamed from R113; footprint (none) -> Resistor_SMD:R_0603_1608Metric
- R138: renamed from R114; footprint (none) -> Resistor_SMD:R_0603_1608Metric
- R139: renamed from R115; footprint (none) -> Resistor_SMD:R_0603_1608Metric
- Y102: renamed from Y101; value Crystal -> 32K; footprint (none) -> Crystal:Crystal_SMD_5032-2Pin_5.0x3.2mm; Manufacturer PN FC-135 32.7680KA-AC0 -> Q13FC1350000300
- renumbered R102 to R142, R106 to R143, R101 to R144, R103 to R145, U102 to U109
Connections:
- net labels added: +3V3, 12V_Sense, BOOT0, BOOT1, CAN_RX, CAN_TX, HV_GRID, IND_DIM, JTCK, JTDI, JTDO, JTMS, LED1, LED2, STP-IN1, STP-IN2, STP-IN3, STP-IN4, STP-IN5, STP-IN6, STP-IN7, STP-IN8, USB-D+, USB-D-, VFD_FILAMENT_A, VFD_LV_BLANK, VFD_LV_CLK, VFD_LV_MOSI, VFD_LV_STROBE
- net labels removed: RPM, VSS_IN
- wire segments 178 -> 575
- no-connect marks 0 -> 16
Other:
- note added: "10mA@1.2V\n5V - R=380\n12V - R=1080"
- note added: "R for current adjustment.\n"
- note added: "Vout=1.25(1+r2/r1(gnd)\n28 R1=2.2k, r2=47k\n"
- moved on the sheet: BT101, C106, C107, C130, C131, C135, C136, C140, C141, D104, D132, D133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

Commit message: Modified the board.
I noticed I had the TDI and TMS? lines PA14 and PA15 switched. I
modified the schematic and board. They should both match what was
actually created.
Changed lines of the file:
@@
 Text Label 8450 9450 0    50   ~ 0
 JTDO
+Text Label 10300 10650 0    50   ~ 0
+JTDI
 Text Label 10300 10550 0    50   ~ 0
-JTDI
-Text Label 10300 10650 0    50   ~ 0
 JTCK
 Text Label 10300 10450 0    50   ~ 0
@@
 Text Label 12400 11550 0    50   ~ 0
 JTMS
+Text Label 12400 11750 0    50   ~ 0
+JTCK
 Text Label 12400 11650 0    50   ~ 0
-JTCK
-Text Label 12400 11750 0    50   ~ 0
 JTDI
 Text Label 12400 11850 0    50   ~ 0

Commit message: Finished rev 1 of the board, changed motor drivers, moved power supply stouff, fixed programming header layout, added power indication LEDS
Parts:
- C123, C126, C127: value C -> 0.1uF
- C124, C125: value C -> 1uF
- R118: value R -> 59K
- R121: value R -> 2.49K
Other:
- note added: "TIMER4\n"
- note added: "Vout=1.25(1+r2/r1\nR1 goes to GND\n28 R1=2.2k, r2=47k\n30.86v, R1=2.49K, R2=59K\n"
- note removed: "Vout=1.25(1+r2/r1(gnd)\n28 R1=2.2k, r2=47k\n"
